Commit message: imu sensörleri eklendi urdf'ten xacroya geçildi monoped modeli eklendi hexapod modeli düzenlendi monoped ve hexapod için control scriptleri eklendi monoped ve hexapod için launch dosyaları eklendi monoped ve hexapod için config dosyaları eklendi

File: models/hexapod/model.urdf (robot description, URDF)
Before this commit: robot hexapod, 19 links, 18 joints
Links:
- added link imu, mass 0.000001; collision box size=0.02 0.001 0.05; visual box size=0.02 0.001 0.05
Joints:
- added joint imu_joint: type fixed, parent lowerleg_4, child imu, origin xyz=0.4 0.0 0.015 rpy=1.57 0.0 1.57
- joint hfe_joint_6: limit lower=0.3 upper=1.4 effort=200 velocity=1.0 -> lower=0.3 upper=0.3 effort=200 velocity=1.0

Commit message: First update

File: models/hexapod/model.urdf (robot description, URDF)
Before this commit: robot hexapod, 20 links, 19 joints
Joints:
- joint imu_joint: origin xyz=0.4 0.0 0.015 rpy=1.57 0.0 1.57 -> xyz=0.4 0.8 0.8 rpy=1.57 1.57 1.57

File: models/hexapod/xacro/macro.hexapod.xacro (robot description, xacro)
@@ -93,4 +93,5 @@
         <xacro:imu legnumber="5"/>
         <xacro:imu legnumber="6"/>
+        <xacro:base_imu/>
     </xacro:macro>
 </robot>

File: models/hexapod/xacro/macro.imu.xacro (robot description, xacro)
@@ -31,12 +31,20 @@
           <topic>__default_topic__</topic>
           <plugin filename="libgazebo_ros_imu_sensor.so" name="imu_plugin">
-              <topicName>hexapod/sensor/imu_leg_${legnumber}</topicName>
-              <bodyName>imu_link</bodyName>
-              <updateRateHZ>10.0</updateRateHZ>
-              <gaussianNoise>0.0</gaussianNoise>
-              <xyzOffset>0 0 0</xyzOffset>
-              <rpyOffset>0 0 0</rpyOffset>
-              <frameName>imu_link</frameName>
-              <initialOrientationAsReference>false</initialOrientationAsReference>
+            <topicName>hexapod/sensor/imu_leg_${legnumber}</topicName>
+            <bodyName>imu_link</bodyName>
+            <updateRateHZ>10.0</updateRateHZ>
+            <gaussianNoise>0.0</gaussianNoise>
+            <xyzOffset>0 0 0</xyzOffset>
+            <rpyOffset>0 0 0</rpyOffset>
+            <frameName>imu_link</frameName>
+            <initialOrientationAsReference>false</initialOrientationAsReference>
+            <gyroscopeNoiseDensity>0.0003394</gyroscopeNoiseDensity>
+            <gyroscopeRandomWalk>3.8785e-05</gyroscopeRandomWalk>
+            <gyroscopeBiasCorrelationTime>1000.0</gyroscopeBiasCorrelationTime>
+            <gyroscopeTurnOnBiasSigma>0.0087</gyroscopeTurnOnBiasSigma>
+            <accelerometerNoiseDensity>0.004</accelerometerNoiseDensity>
+            <accelerometerRandomWalk>0.006</accelerometerRandomWalk>
+            <accelerometerBiasCorrelationTime>300.0</accelerometerBiasCorrelationTime>
+            <accelerometerTurnOnBiasSigma>0.196</accelerometerTurnOnBiasSigma>
           </plugin>
           <pose>0 0 0 0 0 0</pose>
@@ -46,5 +54,61 @@
         <parent link="tibia_${legnumber}"/>
         <child link="imu_${legnumber}"/>
-        <origin xyz="0.4 0.0 0.015" rpy="1.57 0.0 1.57"/>
+        <origin xyz="0.4 0.015 0.0" rpy="1.57 1.57 1.57"/>
+    </joint>
+</xacro:macro>
+<xacro:macro name="base_imu">
+    <link name="imu_base">
+        <inertial>
+            <mass value="0.000001"/>
+            <inertia ixx="0.0" ixy="0.0" ixz="0.0" iyy="0.0" iyz="0.0" izz="0.0"/>
+        </inertial>
+        <visual>
+            <origin xyz="0.0 0.0 0.0" rpy="0.0 0.0 0.0"/>
+            <geometry>
+                <box size="0.02 0.001 0.05"/>
+            </geometry>
+            <material name="yellow">
+                <color rgba="1.0 1.0 0.0 1.0"/>
+            </material>
+        </visual>
+        <collision>
+            <origin xyz="0.0 0.0 0.0" rpy="0.0 0.0 0.0"/>
+            <geometry>
+                <box size="0.02 0.001 0.05"/>
+            </geometry>
+        </collision>
+    </link>
+    <gazebo reference="imu_base">
+      <material>Gazebo/Yellow</material>
+        <sensor name="imu_sensor" type="imu">
+          <always_on>true</always_on>
+          <update_rate>100</update_rate>
+          <visualize>true</visualize>
+          <topic>__default_topic__</topic>
+          <plugin filename="libgazebo_ros_imu_sensor.so" name="imu_plugin">
+            <topicName>hexapod/sensor/imu_base</topicName>
+            <bodyName>imu_link</bodyName>
+            <updateRateHZ>10.0</updateRateHZ>
+            <gaussianNoise>0.0</gaussianNoise>
+            <xyzOffset>0 0 0</xyzOffset>
+            <rpyOffset>0 0 0</rpyOffset>
+            <frameName>imu_link</frameName>
+            <initialOrientationAsReference>false</initialOrientationAsReference>
+            <gyroscopeNoiseDensity>0.0003394</gyroscopeNoiseDensity>
+            <gyroscopeRandomWalk>3.8785e-05</gyroscopeRandomWalk>
+            <gyroscopeBiasCorrelationTime>1000.0</gyroscopeBiasCorrelationTime>
+            <gyroscopeTurnOnBiasSigma>0.0087</gyroscopeTurnOnBiasSigma>
+            <accelerometerNoiseDensity>0.004</accelerometerNoiseDensity>
+            <accelerometerRandomWalk>0.006</accelerometerRandomWalk>
+            <accelerometerBiasCorrelationTime>300.0</accelerometerBiasCorrelationTime>
+            <accelerometerTurnOnBiasSigma>0.196</accelerometerTurnOnBiasSigma>
+          </plugin>
+          <pose>0 0 0 0 0 0</pose>
+        </sensor>
+    </gazebo>
+    <joint name="base_imu_base" type="fixed">
+        <parent link="base"/>
+        <child link="imu_base"/>
+        <origin xyz="0.4 0 0.2" rpy="1.57 0.0 1.57"/>
     </joint>
 </xacro:macro>
