Commit message: Fix tf oriantation for all joints

File: hex_description/models/hexapod/xacro/hexapod.urdf.xacro (robot description, xacro)
@@ -9,28 +9,34 @@
     <xacro:include filename="$(find hex_description)/models/hexapod/xacro/macro.internal_config.xacro"/>
     <xacro:include filename="$(find hex_description)/models/hexapod/xacro/gazebo.control.xacro"/>
-    <!-- <xacro:leg
+    <xacro:leg
     legnumber="1"
     xyz="0.7 0.435 0.05"
-    rpy="0 0 2.44"/> -->
+    rpy="0 0 3.14"
+    y_joint="-1.0472"/>
      <xacro:leg
     legnumber="2"
     xyz="-0.03 0.59 0.05"
-    rpy="0 0 3.14"/>
-    <!-- <xacro:leg
+    rpy="0 0 3.14"
+    y_joint="0"/>
+    <xacro:leg
     legnumber="3"
     xyz="-0.76 0.39 0.05"
-    rpy="0 0 3.84"/>
+    rpy="0 0 3.14"
+    y_joint="1.0472"/>
     <xacro:leg
     legnumber="4"
     xyz="-0.77 -0.345 0.05"
-    rpy="0 0 -0.7"/>
+    rpy="0 0 3.14"
+    y_joint="2.09"/>
     <xacro:leg
     legnumber="5"
     xyz="-0.054 -0.565 0.05"
-    rpy="0 0 0"/>
+    rpy="0 0 3.14"
+    y_joint="3.14"/>
     <xacro:leg
     legnumber="6"
     xyz="0.69 -0.435 0.05"
-    rpy="0 0 0.7"/> -->
+    rpy="0 0 3.14"
+    y_joint="4.18"/>
     <xacro:dsr_config_coeff_base/>
 </robot>

File: hex_description/models/hexapod/xacro/macro.leg.urdf.xacro (robot description, xacro)
@@ -1,5 +1,5 @@
 <?xml version="1.0"?>
 <robot xmlns:xacro="http://www.ros.org/wiki/xacro">
-    <xacro:macro name="leg" params="legnumber xyz rpy">
+    <xacro:macro name="leg" params="legnumber xyz rpy y_joint">
         <link name="coxa_${legnumber}">
             <visual>
@@ -14,8 +14,8 @@
             </inertial>
             <collision>
-            <geometry>
-                <mesh filename="package://hex_description/models/hexapod/meshes/coxa.stl" scale="0.01 0.01 0.01"/>
+                <geometry>
+                    <mesh filename="package://hex_description/models/hexapod/meshes/coxa.stl" scale="0.01 0.01 0.01"/>
+                </geometry>
                 <origin xyz="0 0 0" rpy="${rpy}"/>
-            </geometry>
             </collision>
         </link>
@@ -32,8 +32,8 @@
             </inertial>
             <collision>
-            <geometry>
-                <mesh filename="package://hex_description/models/hexapod/meshes/femur.stl" scale="0.01 0.01 0.01"/>
-                <origin xyz="0 0 0" rpy="0 0 3.14"/>
-            </geometry>
+                <geometry>
+                    <mesh filename="package://hex_description/models/hexapod/meshes/femur.stl" scale="0.01 0.01 0.01"/>
+                </geometry>
+                <origin xyz="0 0 0" rpy="1.57 1.57 3.14"/>
             </collision>
         </link>
@@ -43,5 +43,5 @@
                 <mesh filename="package://hex_description/models/hexapod/meshes/tibia.stl" scale="0.01 0.01 0.01"/>
             </geometry>
-            <origin xyz="0 0 0" rpy="0 1.57 0"/>
+            <origin xyz="0 0 0" rpy="0 1.57 1.57"/>
             <material name="tibia"/>
             </visual>
@@ -52,6 +52,6 @@
             <geometry>
                 <mesh filename="package://hex_description/models/hexapod/meshes/tibia.stl" scale="0.01 0.01 0.01"/>
-                <origin xyz="0 0 0" rpy="0 1.57 0"/>
             </geometry>
+            <origin xyz="0 0 0" rpy="0 1.57 1.57"/>
             </collision>
         </link>
@@ -60,5 +60,5 @@
             <parent link="body_bottom"/>
             <child link="coxa_${legnumber}"/>
-            <origin rpy="0 0 0" xyz="${xyz}"/>
+            <origin rpy="0 0 ${y_joint}" xyz="${xyz}"/>
             <limit effort="${base_coxa_effort}" lower="${lower_bc}" upper="${upper_bc}" velocity="${base_coxa_velocity}"/>
             <axis xyz="0 0 1"/>
@@ -84,5 +84,5 @@
             <parent link="tibia_${legnumber}"/>
             <child link="end_point_${legnumber}"/>
-            <origin rpy="0 0.0 0.0" xyz="0 -0.755 0.0"/>
+            <origin rpy="0 0.0 0.0" xyz="0.755 0 0.0"/>
         </joint>
     	<xacro:leg_transmissions legnumber="${legnumber}"/>

File: hex_description/models/hexapod/xacro/propertys.xacro (robot description, xacro)
@@ -17,6 +17,8 @@
     <xacro:property name="upper_cf" value="0.707"/>
     <!-- Femur to tibia joints limits -->
-    <xacro:property name="lower_ft" value="0.707"/>
-    <xacro:property name="upper_ft" value="2.3"/>
+    <!-- <xacro:property name="lower_ft" value="0.707"/>
+    <xacro:property name="upper_ft" value="2.3"/> -->
+    <xacro:property name="lower_ft" value="0"/>
+    <xacro:property name="upper_ft" value="6.28"/>
     <!-- joints stiffness -->
     <xacro:property name="base_coxa_damping" value="60.0"/>
