Commit message: Fix intertia, add F.kinematics , add controller

File: hex_description/models/hexapod/xacro/macro.internal_config.xacro (robot description, xacro)
@@ -3,6 +3,6 @@
     <xacro:macro name="dsr_config_coeff_base">
         <gazebo reference="body_bottom">
-            <kp>1000000.0</kp>
-            <kd>100.0</kd>
+            <kp>10.0</kp>
+            <kd>1.0</kd>
             <mu1>0.5</mu1>
             <mu2>0.5</mu2>
@@ -45,7 +45,7 @@
             <kp>50000.0</kp>
             <kd>1.0</kd>
-            <!-- <minDepth>0.001</minDepth> -->
-            <!-- <maxVel>0.1</maxVel>
-            <fdir1>1 0 0</fdir1> -->
+            <minDepth>0.001</minDepth>
+            <maxVel>0.1</maxVel>
+            <!-- <fdir1>1 0 0</fdir1> -->
             <material>Gazebo/Green</material>
         </gazebo>
@@ -55,7 +55,7 @@
             <kp>50000.0</kp>
             <kd>1.0</kd>
-            <!-- <minDepth>0.001</minDepth> -->
-            <!-- <maxVel>0.1</maxVel>
-            <fdir1>1 0 0</fdir1> -->
+            <minDepth>0.001</minDepth>
+            <maxVel>0.1</maxVel>
+            <!-- <fdir1>1 0 0</fdir1> -->
             <material>Gazebo/Orange</material>
         </gazebo>
@@ -65,7 +65,7 @@
             <kp>50000.0</kp>
             <kd>1.0</kd>
-            <!-- <minDepth>0.001</minDepth> -->
-            <!-- <maxVel>0.1</maxVel>
-            <fdir1>1 0 0</fdir1> -->
+            <minDepth>0.001</minDepth>
+            <maxVel>0.1</maxVel>
+            <!-- <fdir1>1 0 0</fdir1> -->
             <material>Gazebo/Blue</material>
         </gazebo>

File: hex_description/models/hexapod/xacro/macro.leg.urdf.xacro (robot description, xacro)
@@ -12,4 +12,5 @@
             <inertial>
               <xacro:box_inertia m="${coxa_mass}" x="0.15" y="0.5" z="0.5"/>
+              <origin xyz="0 0 0" rpy="${rpy}"/>
             </inertial>
             <collision>
@@ -30,4 +31,5 @@
             <inertial>
                  <xacro:box_inertia m="${femur_mass}" x="0.45" y="0.72" z="0.17"/>
+                 <origin xyz="0 0 0" rpy="1.57 1.57 1.57"/>
             </inertial>
             <collision>
@@ -40,11 +42,12 @@
         <link name="tibia_${legnumber}">
             <visual>
-            <geometry>
-                <mesh filename="package://hex_description/models/hexapod/meshes/tibia.stl" scale="0.01 0.01 0.01"/>
-            </geometry>
-            <origin xyz="0 0 0" rpy="0 1.57 1.57"/>
-            <material name="tibia"/>
+                <geometry>
+                    <mesh filename="package://hex_description/models/hexapod/meshes/tibia.stl" scale="0.01 0.01 0.01"/>
+                </geometry>
+                <origin xyz="0 0 0" rpy="0 1.57 1.57"/>
+                <material name="tibia"/>
             </visual>
             <inertial>
+                <origin xyz="0 0 0" rpy="0 1.57 0"/>
                 <xacro:box_inertia m="${femur_mass}" x="0.3" y="1.15" z="0.22"/>
             </inertial>

File: hex_description/models/hexapod/xacro/propertys.xacro (robot description, xacro)
@@ -17,8 +17,8 @@
     <xacro:property name="upper_cf" value="0.707"/>
     <!-- Femur to tibia joints limits -->
-    <!-- <xacro:property name="lower_ft" value="0.707"/>
-    <xacro:property name="upper_ft" value="2.3"/> -->
-    <xacro:property name="lower_ft" value="0"/>
-    <xacro:property name="upper_ft" value="6.28"/>
+    <xacro:property name="lower_ft" value="-2.3"/>
+    <xacro:property name="upper_ft" value="0"/>
+    <!-- <xacro:property name="lower_ft" value="0"/>
+    <xacro:property name="upper_ft" value="6.28"/> -->
     <!-- joints stiffness -->
     <xacro:property name="base_coxa_damping" value="60.0"/>
