Commit message: update xacro files for new model

File: hex_description/models/hexapod/xacro/hexapod.urdf (robot description, URDF)
Before this commit: robot hexapod, 23 links, 22 joints
Links:
- added link end_point_1
- added link end_point_2
- added link end_point_3
- added link end_point_4
- added link end_point_5
- added link end_point_6
- link board_bracket: mass 0.3 -> 0.7
- link body_bottom: mass 0.2 -> 0.6
- link body_top: mass 0.2 -> 0.7
- link cover_top: mass 0.05 -> 0.1
- link coxa_1: mass 0.2 -> 0.6
- link coxa_2: mass 0.2 -> 0.6
- link coxa_3: mass 0.2 -> 0.6
- link coxa_4: mass 0.2 -> 0.6
- link coxa_5: mass 0.2 -> 0.6
- link coxa_6: mass 0.2 -> 0.6
- link femur_1: mass 0.2 -> 0.6
- link femur_2: mass 0.2 -> 0.6
- link femur_3: mass 0.2 -> 0.6
- link femur_4: mass 0.2 -> 0.6
- link femur_5: mass 0.2 -> 0.6
- link femur_6: mass 0.2 -> 0.6
- link tibia_1: mass 0.2 -> 0.6
- link tibia_2: mass 0.2 -> 0.6
- link tibia_3: mass 0.2 -> 0.6
- link tibia_4: mass 0.2 -> 0.6
- link tibia_5: mass 0.2 -> 0.6
- link tibia_6: mass 0.2 -> 0.6
Joints:
- added joint end_point_joint_1: type fixed, parent tibia_1, child end_point_1, origin xyz=0.755 0 0.0 rpy=0 0.0 0.0
- added joint end_point_joint_2: type fixed, parent tibia_2, child end_point_2, origin xyz=0.755 0 0.0 rpy=0 0.0 0.0
- added joint end_point_joint_3: type fixed, parent tibia_3, child end_point_3, origin xyz=0.755 0 0.0 rpy=0 0.0 0.0
- added joint end_point_joint_4: type fixed, parent tibia_4, child end_point_4, origin xyz=0.755 0 0.0 rpy=0 0.0 0.0
- added joint end_point_joint_5: type fixed, parent tibia_5, child end_point_5, origin xyz=0.755 0 0.0 rpy=0 0.0 0.0
- added joint end_point_joint_6: type fixed, parent tibia_6, child end_point_6, origin xyz=0.755 0 0.0 rpy=0 0.0 0.0
- joint base_coxa_joint_1: limit lower=-0.707 upper=0.707 effort=50.0 velocity=1 -> lower=-0.707 upper=0.707 effort=50.0 velocity=1.0; origin xyz=0.7 0.435 0.05 rpy=0 0 2.44 -> xyz=0.7 0.435 0.05 rpy=0 0 -1.0472
- joint base_coxa_joint_2: limit lower=-0.707 upper=0.707 effort=50.0 velocity=1 -> lower=-0.707 upper=0.707 effort=50.0 velocity=1.0; origin xyz=-0.03 0.59 0.05 rpy=0 0 3.14 -> xyz=-0.03 0.59 0.05 rpy=0 0 0
- joint base_coxa_joint_3: limit lower=-0.707 upper=0.707 effort=50.0 velocity=1 -> lower=-0.707 upper=0.707 effort=50.0 velocity=1.0; origin xyz=-0.76 0.39 0.05 rpy=0 0 3.84 -> xyz=-0.76 0.39 0.05 rpy=0 0 1.0472
- joint base_coxa_joint_4: limit lower=-0.707 upper=0.707 effort=50.0 velocity=1 -> lower=-0.707 upper=0.707 effort=50.0 velocity=1.0; origin xyz=-0.77 -0.345 0.05 rpy=0 0 -0.7 -> xyz=-0.77 -0.345 0.05 rpy=0 0 2.09
- joint base_coxa_joint_5: limit lower=-0.707 upper=0.707 effort=50.0 velocity=1 -> lower=-0.707 upper=0.707 effort=50.0 velocity=1.0; origin xyz=-0.054 -0.565 0.05 rpy=0 0 0 -> xyz=-0.054 -0.565 0.05 rpy=0 0 3.14
- joint base_coxa_joint_6: limit lower=-0.707 upper=0.707 effort=50.0 velocity=1 -> lower=-0.707 upper=0.707 effort=50.0 velocity=1.0; origin xyz=0.69 -0.435 0.05 rpy=0 0 0.7 -> xyz=0.69 -0.435 0.05 rpy=0 0 4.18
- joint coxa_femur_joint_1: axis 1 0 0 -> 0 0 1; limit lower=-0.707 upper=0.707 effort=200.0 velocity=1 -> lower=-0.707 upper=0.707 effort=50.0 velocity=1.0; origin xyz=0.09 -0.345 -0.04 rpy=0.0 0.0 0.0 -> xyz=-0.09 0.345 -0.04 rpy=-1.57 3.14 -1.57
- joint coxa_femur_joint_2: axis 1 0 0 -> 0 0 1; limit lower=-0.707 upper=0.707 effort=200.0 velocity=1 -> lower=-0.707 upper=0.707 effort=50.0 velocity=1.0; origin xyz=0.09 -0.345 -0.04 rpy=0.0 0.0 0.0 -> xyz=-0.09 0.345 -0.04 rpy=-1.57 3.14 -1.57
- joint coxa_femur_joint_3: axis 1 0 0 -> 0 0 1; limit lower=-0.707 upper=0.707 effort=200.0 velocity=1 -> lower=-0.707 upper=0.707 effort=50.0 velocity=1.0; origin xyz=0.09 -0.345 -0.04 rpy=0.0 0.0 0.0 -> xyz=-0.09 0.345 -0.04 rpy=-1.57 3.14 -1.57
- joint coxa_femur_joint_4: axis 1 0 0 -> 0 0 1; limit lower=-0.707 upper=0.707 effort=200.0 velocity=1 -> lower=-0.707 upper=0.707 effort=50.0 velocity=1.0; origin xyz=0.09 -0.345 -0.04 rpy=0.0 0.0 0.0 -> xyz=-0.09 0.345 -0.04 rpy=-1.57 3.14 -1.57
- joint coxa_femur_joint_5: axis 1 0 0 -> 0 0 1; limit lower=-0.707 upper=0.707 effort=200.0 velocity=1 -> lower=-0.707 upper=0.707 effort=50.0 velocity=1.0; origin xyz=0.09 -0.345 -0.04 rpy=0.0 0.0 0.0 -> xyz=-0.09 0.345 -0.04 rpy=-1.57 3.14 -1.57
- joint coxa_femur_joint_6: axis 1 0 0 -> 0 0 1; limit lower=-0.707 upper=0.707 effort=200.0 velocity=1 -> lower=-0.707 upper=0.707 effort=50.0 velocity=1.0; origin xyz=0.09 -0.345 -0.04 rpy=0.0 0.0 0.0 -> xyz=-0.09 0.345 -0.04 rpy=-1.57 3.14 -1.57
- joint femur_tibia_joint_1: axis 1 0 0 -> 0 0 1; limit lower=0.707 upper=2.3 effort=200.0 velocity=1 -> lower=-2.3 upper=0 effort=50.0 velocity=1.0; origin xyz=-0.035 -0.555 0.0 rpy=0 0.0 0.0 -> xyz=0.555 0.035 0.0 rpy=0 0.0 0.0
- joint femur_tibia_joint_2: axis 1 0 0 -> 0 0 1; limit lower=0.707 upper=2.3 effort=200.0 velocity=1 -> lower=-2.3 upper=0 effort=50.0 velocity=1.0; origin xyz=-0.035 -0.555 0.0 rpy=0 0.0 0.0 -> xyz=0.555 0.035 0.0 rpy=0 0.0 0.0
- joint femur_tibia_joint_3: axis 1 0 0 -> 0 0 1; limit lower=0.707 upper=2.3 effort=200.0 velocity=1 -> lower=-2.3 upper=0 effort=50.0 velocity=1.0; origin xyz=-0.035 -0.555 0.0 rpy=0 0.0 0.0 -> xyz=0.555 0.035 0.0 rpy=0 0.0 0.0
- joint femur_tibia_joint_4: axis 1 0 0 -> 0 0 1; limit lower=0.707 upper=2.3 effort=200.0 velocity=1 -> lower=-2.3 upper=0 effort=50.0 velocity=1.0; origin xyz=-0.035 -0.555 0.0 rpy=0 0.0 0.0 -> xyz=0.555 0.035 0.0 rpy=0 0.0 0.0
- joint femur_tibia_joint_5: axis 1 0 0 -> 0 0 1; limit lower=0.707 upper=2.3 effort=200.0 velocity=1 -> lower=-2.3 upper=0 effort=50.0 velocity=1.0; origin xyz=-0.035 -0.555 0.0 rpy=0 0.0 0.0 -> xyz=0.555 0.035 0.0 rpy=0 0.0 0.0
- joint femur_tibia_joint_6: axis 1 0 0 -> 0 0 1; limit lower=0.707 upper=2.3 effort=200.0 velocity=1 -> lower=-2.3 upper=0 effort=50.0 velocity=1.0; origin xyz=-0.035 -0.555 0.0 rpy=0 0.0 0.0 -> xyz=0.555 0.035 0.0 rpy=0 0.0 0.0
